File: PCB2/PlacaDrivers/PlacaDrivers.sch (KiCad schematic (older format))
At the start: 145 parts, among them U1 TB9051FTG, U2 TB9051FTG, U3 TB9051FTG, U4 TB9051FTG, U5 TB9051FTG, U6 TB9051FTG, U7 TB9051FTG, U8 TB9051FTG

Commit message: Placa driver casi enrutada, step y medidas exportadas
Parts:
- removed C? (x8): 0.47uF, symbol device:C_Small
- removed R? (x9): 1k, symbol device:R_Small
- removed R? (x15): 220, symbol device:R_Small
- removed R? (x7): 10k, symbol device:R_Small
- added C17: 10uF, Capacitors_SMD:C_0805, symbol device:C_Small
- added D1: MMSZ4700-G3-08, Diode_SMD:D_SOD-123, symbol device:D_Zener_Small_ALT
- added JP1: SJ-A0, Jumpers:SMT-JUMPER_2_NO_SILK, symbol device:Jumper_NO_Small
- added JP2: SJ-A1, Jumpers:SMT-JUMPER_2_NO_SILK, symbol device:Jumper_NO_Small
- added JP3: SJ-A2, Jumpers:SMT-JUMPER_2_NO_SILK, symbol device:Jumper_NO_Small
- added JP4: SJ-A3, Jumpers:SMT-JUMPER_2_NO_SILK, symbol device:Jumper_NO_Small
- added JP5: SJ-A4, Jumpers:SMT-JUMPER_2_NO_SILK, symbol device:Jumper_NO_Small
- added JP6: SJ-A5, Jumpers:SMT-JUMPER_2_NO_SILK, symbol device:Jumper_NO_Small
- added P5: HEADER1, Pin_Headers:Pin_Header_Straight_1x15, symbol conn:CONN_01X15
- added P6: HEADER2, Pin_Headers:Pin_Header_Straight_1x15, symbol conn:CONN_01X15
- added P7: MAIN POWER, Connectors_Molex:Molex_Microfit3_Header_02x02_Angled_43045-040x, symbol conn:CONN_02X02
- added Q1: FDD9411L-F085, TO_SOT_Packages_SMD:TO-252-3_TabPin4, symbol SparkFun-DiscreteSemi:MOSFET-NCHANNELFDD8780
- added R1: 20k, Resistors_SMD:R_0603, symbol device:R_Small
- added R2: 1k, Resistors_SMD:R_0603, symbol device:R_Small
- added R21, R22, R23, R24, R25, R26, R45, R70, R79: 10k, Resistors_SMD:R_0603, symbol device:R_Small
- C10, C11, C12, C15, C16, C20, C21, C22, C23, C24, C25, C28, C29, C3, C32, C33, C34, C35, C36, C37, C4, C40, C41, C44, C45, C46, C47, C48, C49, C7, C8, C9: renamed from C?; footprint (none) -> Capacitors_SMD:C_0805
- C18, C19, C30, C31, C42, C43, C5, C6: renamed from C?; footprint (none) -> Capacitors_SMD:c_elec_6.3x4.5
- P1, P10, P11, P12, P2, P3, P4, P9: renamed from P?; footprint (none) -> Connectors_Molex:Molex_Microfit3_Header_02x01_Angled_43045-020x
- R10, R100, R101, R102, R103, R104, R105, R11, R13, R15, R16, R17, R18, R19, R20, R33, R34, R36, R37, R39, R40, R41, R42, R43, R44, R46, R47, R5, R7, R71, R72, R74, R75, R77, R78, R8, R80, R81, R82, R83, R84, R85, R9, R92, R93, R95, R96, R98, R99: renamed from R?; footprint (none) -> Resistors_SMD:R_0603
- U1, U2, U3, U4, U5, U6, U7, U8: footprint (none) -> frizzy_ics:QFN-28-1EP_6x6mm_Pitch0.65mm
- U9: renamed from U?; footprint TSSOP28 -> Silicon-Standard:TSSOP28
Connections:
- net ENB_2 is gone; now on net ENB: R33.2
- net ENB_3 is gone; now on net ENB: R74.2
- net ENB_4 is gone; now on net ENB: R95.2
- net ENB_5 is gone; now on net ENB: R7.2
- net ENB_6 is gone; now on net ENB: R36.2
- net ENB_7 is gone; now on net ENB: R71.2
- net ENB_8 is gone; now on net ENB: R92.2
- net EN_2 is gone; now on net EN: R41.2
- net EN_3 is gone; now on net EN: R82.2
- net EN_4 is gone; now on net EN: R102.2
- net EN_5 is gone; now on net EN: R15.2
- net EN_6 is gone; now on net EN: R43.2
- net EN_7 is gone; now on net EN: R80.2
- net EN_8 is gone; now on net EN: R100.2
- net OCC_2 is gone; now on net VCC: R39.2
- net OCC_3 is gone; now on net VCC: R78.2
- net OCC_4 is gone; now on net VCC: R99.2
- net OCC_5 is gone; now on net VCC: R13.2
- net OCC_6 is gone; now on net VCC: R40.2
- net OCC_7 is gone; now on net VCC: R77.2
- net OCC_8 is gone; now on net VCC: R98.2
- net GND: now also U9.14 (GND), U9.25 (EXTCLK), C17.2, D1.2 (A), P5.4 (P4), P6.2 (P2), Q1.3 (S), R21.2, R22.2, R23.2, R24.2, R25.2, R26.2, R45.1
- net PWM1_1: now also U9.6 (PWM0)
- net PWM1_2: now also U9.8 (PWM2)
- net PWM1_3: now also U9.10 (PWM4)
- net PWM1_4: now also U9.12 (PWM6)
- net PWM1_5: now also U9.15 (PWM8)
- net PWM1_6: now also U9.17 (PWM10)
- net PWM1_7: now also U9.19 (PWM12)
- net PWM1_8: now also U9.21 (PWM14)
- net PWM2_1: now also U9.7 (PWM1)
- net PWM2_2: now also U9.9 (PWM3)
- net PWM2_3: now also U9.11 (PWM5)
- net PWM2_4: now also U9.13 (PWM7)
- net PWM2_5: now also U9.16 (PWM9)
- net PWM2_6: now also U9.18 (PWM11)
- net PWM2_7: now also U9.20 (PWM13)
- net PWM2_8: now also U9.22 (PWM15)
- net VCC: now also U9.28 (VDD), C17.1, JP1.1, JP2.1, JP3.1, JP4.1, JP5.1, JP6.1, P6.4 (P4), R2.2, R70.1, R79.1
- net VIN: now also P7.1 (P1), P7.3 (P3), R1.1
- net at U1.1 (OCC): now also R2.1
- net DIAG: now reaches U1.18 (DIAG)
- net DIAG: now also R5.1, R9.2, U2.18 (DIAG), U3.18 (DIAG), U4.18 (DIAG), U5.18 (DIAG), U6.18 (DIAG), U7.18 (DIAG), U8.18 (DIAG)
- net A0: now reaches U9.1 (A0)
- net A0: now also JP1.2, R26.1
- net A1: now reaches U9.2 (A1)
- net A1: now also JP2.2, R25.1
- net OE: now reaches U9.23 (#OE)
- net OE: now also P5.9 (P9), R45.2
- net A5: now reaches U9.24 (A5)
- net A5: now also JP6.2, R21.1
- net SCL: now reaches U9.26 (SCL)
- net SCL: now also P6.7 (P7), R70.2
- net SDA: now reaches U9.27 (SDA)
- net SDA: now also P6.8 (P8), R79.2
- net A2: now reaches U9.3 (A2)
- net A2: now also JP3.2, R24.1
- net A3: now reaches U9.4 (A3)
- net A3: now also JP4.2, R23.1
- net A4: now reaches U9.5 (A4)
- net A4: now also JP5.2, R22.1
- net DIAG_5 renamed DIAG_READ
- net DIAG_READ: now also P5.10 (P10)
- net ENB_1 renamed ENB
- net ENB: now also P5.8 (P8)
- net EN_1 renamed EN
- net EN: now also P5.7 (P7)
- new net: D1.1 (K), Q1.1 (G), R1.2
- new net GNDA: P7.2 (P2), P7.4 (P4), Q1.4 (D)
- no-connect marks 24 -> 54
Other:
- note added: "+12V"
- note added: "+5V"
- note added: "A0"
- note added: "A1"
- note added: "A2"
- note added: "A3"
- note added: "A4"
- note added: "A5"
- note added: "A6"
- note added: "A7"
- note added: "AREF"
- note added: "D10"
- note added: "D11-MOSI"
- note added: "D12-MISO"
- note added: "D13-SCK"
- note added: "D2"
- note added: "D3"
- note added: "D4"
- note added: "D5"
- note added: "D6"
- note added: "D7"
- note added: "D8"
- note added: "D9"
- note added: "GND"
- note added: "NC"
- note added: "RST"
- note added: "RXD"
- note added: "TXD"
- moved on the sheet: R5, R9, U9

Commit message: Documentos de referencia actualizados
Parts:
- Q1: symbol SparkFun-DiscreteSemi:MOSFET-NCHANNELFDD8780 -> PlacaDrivers-rescue:MOSFET-NCHANNELFDD8780-SparkFun-DiscreteSemi
Changed lines of the file:
@@
 $EndComp
 $Comp
-L SparkFun-DiscreteSemi:MOSFET-NCHANNELFDD8780 Q1
+L PlacaDrivers-rescue:MOSFET-NCHANNELFDD8780-SparkFun-DiscreteSemi Q1
 U 1 1 61BB4484
 P 15700 11200
