File: PCB4/PlacaDynamixel/PlacaDynamixel.kicad_pcb (KiCad board)
At the start: 2 copper layers, 49 x 55.2 mm, 18 parts, among them P1 CONN_01X03, P2 CONN_01X03, P3 PWR-Servo, P4 CONN_01X03, P5 CONN_01X03, P6 HEADER1, P7 HEADER2, Q1 FDD9411L-f085, U1 74LS241

Commit message: Documentos de referencia actualizados
Parts:
- added G***: LOGO, logos_frizzy:logoWTF_small, F.Cu at (133.2, 93.8)
- moved D1 50.3 mm to (142.4, 97.8)
- moved JP1 50.3 mm to (128.2, 72.6)
- moved JP2 50.3 mm to (128.2, 75.2)
- moved P1 50.3 mm to (158.2, 73.2)
- moved P2 50.3 mm to (134.8, 73.2)
- moved P3 50.3 mm to (145.8, 109.3)
- moved P4 50.3 mm to (150.3, 73.2)
- moved P6 50.3 mm to (125.2, 72.7)
- moved Q1 50.3 mm to (150.4, 97.1)
- moved R1 50.3 mm to (151.2, 77.2)
- moved R2 50.3 mm to (139.9, 97.1)
- moved REF** 50.3 mm to (166.4, 114.6)
- moved REF** 50.3 mm to (166.4, 67.6)
- moved U1 50.3 mm to (145.8, 84.8)
- moved REF** 50.3 mm to (125.2, 67.6)
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Other:
- board size 49 x 55.2 mm -> 49 x 55.3 mm
- board text added: "+"
- board text added: "DATA"
- board text added: "GND"
- board text added: "PlacaDynamixel V0.1"
- board text added: "VDD"
