File: PCB4/PlacaDynamixel/PlacaDynamixel.sch (KiCad schematic (older format))
At the start: 14 parts, among them P1 CONN_01X03, P2 CONN_01X03, P3 PWR-Servo, P4 CONN_01X03, P5 CONN_01X03, P6 HEADER1, P7 HEADER2, Q1 FDD9411L-f085, U1 74LS241

Commit message: Documentos de referencia actualizados
Parts:
- Q1: symbol SparkFun-DiscreteSemi:MOSFET-NCHANNELFDD8780 -> PlacaDynamixel-rescue:MOSFET-NCHANNELFDD8780-SparkFun-DiscreteSemi
Changed lines of the file:
@@
 NoConn ~ 3850 3150
 $Comp
-L SparkFun-DiscreteSemi:MOSFET-NCHANNELFDD8780 Q1
+L PlacaDynamixel-rescue:MOSFET-NCHANNELFDD8780-SparkFun-DiscreteSemi Q1
 U 1 1 600E41E2
 P 6550 5350
